File: KiCad/pwrsup.kicad_sch (KiCad schematic)
At the start: 16 parts, among them U1 L7805, U6 TLE2426xP, U7 TLE2426xP, U8 TLE2426xP

Commit message: Some TP -> Headers, added footprints, fixed battery footprint, started layout of board.
Parts:
- added TP3: 4.5V, TestPoint:TestPoint_Pad_D2.0mm, symbol Connector:TestPoint_Small
- C1: renamed from C5; footprint (none) -> Capacitor_THT:CP_Radial_D5.0mm_P2.00mm
- C4: renamed from C3; footprint (none) -> Capacitor_THT:CP_Radial_D5.0mm_P2.00mm
- C5: renamed from C4; footprint (none) -> Capacitor_THT:CP_Radial_D5.0mm_P2.00mm
- TP1: renamed from TP4; footprint (none) -> TestPoint:TestPoint_Pad_D2.0mm
- TP2: renamed from TP3; footprint (none) -> TestPoint:TestPoint_Pad_D2.0mm
- TP4: renamed from TP1; footprint (none) -> TestPoint:TestPoint_Pad_D2.0mm
- TP5: renamed from TP2; footprint (none) -> TestPoint:TestPoint_Pad_D2.0mm
- TP6: renamed from TP7; footprint (none) -> TestPoint:TestPoint_Pad_D2.0mm
- TP7: renamed from TP8; footprint (none) -> TestPoint:TestPoint_Pad_D2.0mm
- renumbered C1 to C2, C2 to C3, U8 to U1, U1 to U2, U6 to U3, U7 to U4
Connections:
- net VDIV: now also TP3.1
Other:
- moved on the sheet: TP2
Changed lines of the file:
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@@
 	(paper "A4")
+	(junction
+		(at 67.31 60.96)
+		(diameter 0)
+		(color 0 0 0 0)
+	)
 	(junction
 		(at 220.98 60.96)
@@
 	)
 	(junction
-		(at 52.07 21.59)
-		(diameter 0)
-		(color 0 0 0 0)
-	)
-	(junction
 		(at 68.58 39.37)
 		(diameter 0)
@@
 	)
 	(junction
+		(at 48.26 21.59)
+		(diameter 0)
+		(color 0 0 0 0)
+	)
+	(junction
 		(at 55.88 21.59)
 		(diameter 0)
@@
 	(wire
 		(pts
+			(xy 67.31 60.96) (xy 60.96 60.96)
+		)
+		(stroke
+			(width 0)
+			(type default)
+		)
+	)
+	(wire
+		(pts
 			(xy 220.98 60.96) (xy 214.63 60.96)
 		)
@@
 	(wire
 		(pts
-			(xy 77.47 60.96) (xy 60.96 60.96)
+			(xy 77.47 60.96) (xy 67.31 60.96)
 		)
 		(stroke
@@
 	(wire
 		(pts
+			(xy 48.26 21.59) (xy 55.88 21.59)
+		)
+		(stroke
+			(width 0)
+			(type default)
+		)
+	)
+	(wire
+		(pts
 			(xy 189.23 63.5) (xy 187.96 63.5)
 		)
@@
 	(wire
 		(pts
-			(xy 34.29 21.59) (xy 52.07 21.59)
+			(xy 34.29 21.59) (xy 48.26 21.59)
 		)
 		(stroke
@@
 		(pts
 			(xy 43.18 39.37) (xy 55.88 39.37)
-		)
-		(stroke
-			(width 0)
-			(type default)
-		)
-	)
-	(wire
-		(pts
-			(xy 52.07 21.59) (xy 55.88 21.59)
 		)
 		(stroke
@@
 		(on_board yes)
 		(dnp no)
-		(property "Reference" "TP7"
+		(property "Reference" "TP6"
 			(at 148.59 66.04 90)
 			(effects
@@
 			)
 		)
-		(property "Footprint" ""
+		(property "Footprint" "TestPoint:TestPoint_Pad_D2.0mm"
 			(at 148.59 66.04 0)
 			(effects
@@
 			(project "ChipTester_354"
 				(path "/57b9e980-cd8f-44e4-af61-2cbd5bb30325/462ebe9c-fcaa-4c45-9d51-a2484be3186e"
-					(reference "TP7")
+					(reference "TP6")
 					(unit 1)
 				)
@@
 		(on_board yes)
 		(dnp no)
-		(property "Reference" "C3"
+		(property "Reference" "C4"
 			(at 102.87 74.9238 0)
 			(effects
@@
 			)
 		)
-		(property "Footprint" ""
+		(property "Footprint" "Capacitor_THT:CP_Radial_D5.0mm_P2.00mm"
 			(at 105.41 73.66 0)
 			(effects
@@
 			(project "ChipTester_354"
 				(path "/57b9e980-cd8f-44e4-af61-2cbd5bb30325/462ebe9c-fcaa-4c45-9d51-a2484be3186e"
-					(reference "C3")
+					(reference "C4")
+					(unit 1)
+				)
+			)
+		)
+	)
+	(symbol
+		(lib_id "Connector:TestPoint_Small")
+		(at 67.31 60.96 90)
+		(unit 1)
+		(exclude_from_sim no)
+		(in_bom yes)
+		(on_board yes)
+		(dnp no)
+		(fields_autoplaced yes)
+		(property "Reference" "TP3"
+			(at 67.31 55.88 90)
+			(effects
+				(font
+					(size 1.27 1.27)
+				)
+			)
+		)
+		(property "Value" "4.5V"
+			(at 67.31 58.42 90)
+			(effects
+				(font
+					(size 1.27 1.27)
+				)
+			)
+		)
+		(property "Footprint" "TestPoint:TestPoint_Pad_D2.0mm"
+			(at 67.31 55.88 0)
+			(effects
+				(font
+					(size 1.27 1.27)
+				)
+				(hide yes)
+			)
+		)
+		(property "Datasheet" "~"
+			(at 67.31 55.88 0)
+			(effects
+				(font
+					(size 1.27 1.27)
+				)
+				(hide yes)
+			)
+		)
+		(property "Description" "test point"
+			(at 67.31 60.96 0)
+			(effects
+				(font
+					(size 1.27 1.27)
+				)
+				(hide yes)
+			)
+		)
+		(pin "1"
+		)
+		(instances
+			(project "ChipTester_354"
+				(path "/57b9e980-cd8f-44e4-af61-2cbd5bb30325/462ebe9c-fcaa-4c45-9d51-a2484be3186e"
+					(reference "TP3")
 					(unit 1)
 				)
@@
 		(dnp no)
 		(fields_autoplaced yes)
-		(property "Reference" "U6"
+		(property "Reference" "U3"
 			(at 119.38 53.34 0)
 			(effects
@@
 			(project ""
 				(path "/57b9e980-cd8f-44e4-af61-2cbd5bb30325/462ebe9c-fcaa-4c45-9d51-a2484be3186e"
-					(reference "U6")
+					(reference "U3")
 					(unit 1)
 				)
@@
 		(dnp no)
 		(fields_autoplaced yes)
-		(property "Reference" "TP4"
+		(property "Reference" "TP1"
 			(at 44.45 38.0999 0)
 			(effects
@@
 			)
 		)
-		(property "Footprint" ""
+		(property "Footprint" "TestPoint:TestPoint_Pad_D2.0mm"
 			(at 48.26 39.37 0)
 			(effects
@@
 			(project ""
 				(path "/57b9e980-cd8f-44e4-af61-2cbd5bb30325/462ebe9c-fcaa-4c45-9d51-a2484be3186e"
-					(reference "TP4")
+					(reference "TP1")
 					(unit 1)
 				)
@@
 		(dnp no)
 		(fields_autoplaced yes)
-		(property "Reference" "U1"
+		(property "Reference" "U2"
 			(at 68.58 15.24 0)
 			(effects
@@
 			(project ""
 				(path "/57b9e980-cd8f-44e4-af61-2cbd5bb30325/462ebe9c-fcaa-4c45-9d51-a2484be3186e"
-					(reference "U1")
+					(reference "U2")
 					(unit 1)
 				)
@@
 		(on_board yes)
 		(dnp no)
-		(property "Reference" "C2"
+		(property "Reference" "C3"
 			(at 77.47 29.2162 0)
 			(effects
@@
 			(project "ChipTester_354"
 				(path "/57b9e980-cd8f-44e4-af61-2cbd5bb30325/462ebe9c-fcaa-4c45-9d51-a2484be3186e"
-					(reference "C2")
+					(reference "C3")
 					(unit 1)
 				)
@@
 		(dnp no)
 		(fields_autoplaced yes)
-		(property "Reference" "TP1"
+		(property "Reference" "TP4"
 			(at 86.36 16.51 90)
 			(effects
@@
 			)
 		)
-		(property "Footprint" ""
+		(property "Footprint" "TestPoint:TestPoint_Pad_D2.0mm"
 			(at 86.36 16.51 0)
 			(effects
@@
 			(project ""
 				(path "/57b9e980-cd8f-44e4-af61-2cbd5bb30325/462ebe9c-fcaa-4c45-9d51-a2484be3186e"
-					(reference "TP1")
+					(reference "TP4")
 					(unit 1)
 				)
@@
 		(on_board yes)
 		(dnp no)
-		(property "Reference" "C4"
+		(property "Reference" "C5"
 			(at 185.42 74.9238 0)
 			(effects
@@
 			)
 		)
-		(property "Footprint" ""
+		(property "Footprint" "Capacitor_THT:CP_Radial_D5.0mm_P2.00mm"
 			(at 187.96 73.66 0)
 			(effects
@@
 			(project "ChipTester_354"
 				(path "/57b9e980-cd8f-44e4-af61-2cbd5bb30325/462ebe9c-fcaa-4c45-9d51-a2484be3186e"
-					(reference "C4")
+					(reference "C5")
 					(unit 1)
 				)
@@
 		(on_board yes)
 		(dnp no)
-		(property "Reference" "TP8"
+		(property "Reference" "TP7"
 			(at 222.2501 62.23 90)
 			(effects
@@
 			)
 		)
-		(property "Footprint" ""
+		(property "Footprint" "TestPoint:TestPoint_Pad_D2.0mm"
 			(at 226.06 60.96 0)
 			(effects
@@
 			(project "ChipTester_354"
 				(path "/57b9e980-cd8f-44e4-af61-2cbd5bb30325/462ebe9c-fcaa-4c45-9d51-a2484be3186e"
-					(reference "TP8")
+					(reference "TP7")
 					(unit 1)
 				)
@@
 		(on_board yes)
 		(dnp no)
-		(property "Reference" "C5"
+		(property "Reference" "C1"
 			(at 29.21 72.3838 0)
 			(effects
@@
 			)
 		)
-		(property "Footprint" ""
+		(property "Footprint" "Capacitor_THT:CP_Radial_D5.0mm_P2.00mm"
 			(at 31.75 71.12 0)
 			(effects
@@
 			(project "ChipTester_354"
 				(path "/57b9e980-cd8f-44e4-af61-2cbd5bb30325/462ebe9c-fcaa-4c45-9d51-a2484be3186e"
-					(reference "C5")
+					(reference "C1")
 					(unit 1)
 				)
@@
 		(dnp no)
 		(fields_autoplaced yes)
-		(property "Reference" "C1"
+		(property "Reference" "C2"
 			(at 58.42 29.2162 0)
 			(effects
@@
 			(project ""
 				(path "/57b9e980-cd8f-44e4-af61-2cbd5bb30325/462ebe9c-fcaa-4c45-9d51-a2484be3186e"
-					(reference "C1")
+					(reference "C2")
 					(unit 1)
 				)
@@
 		(dnp no)
 		(fields_autoplaced yes)
-		(property "Reference" "U8"
+		(property "Reference" "U1"
 			(at 48.26 53.34 0)
 			(effects
@@
 			(project "ChipTester_354"
 				(path "/57b9e980-cd8f-44e4-af61-2cbd5bb30325/462ebe9c-fcaa-4c45-9d51-a2484be3186e"
-					(reference "U8")
+					(reference "U1")
 					(unit 1)
 				)
@@
 		(dnp no)
 		(fields_autoplaced yes)
-		(property "Reference" "TP2"
+		(property "Reference" "TP5"
 			(at 86.36 34.29 90)
 			(effects
@@
 			)
 		)
-		(property "Footprint" ""
+		(property "Footprint" "TestPoint:TestPoint_Pad_D2.0mm"
 			(at 86.36 34.29 0)
 			(effects
@@
 			(project "ChipTester_354"
 				(path "/57b9e980-cd8f-44e4-af61-2cbd5bb30325/462ebe9c-fcaa-4c45-9d51-a2484be3186e"
-					(reference "TP2")
+					(reference "TP5")
 					(unit 1)
 				)
@@
 	(symbol
 		(lib_id "Connector:TestPoint_Small")
-		(at 52.07 21.59 90)
+		(at 48.26 21.59 90)
 		(unit 1)
 		(exclude_from_sim no)
@@
 		(dnp no)
 		(fields_autoplaced yes)
-		(property "Reference" "TP3"
-			(at 52.07 16.51 90)
+		(property "Reference" "TP2"
+			(at 48.26 16.51 90)
 			(effects
 				(font
@@
 		)
 		(property "Value" "VBATT+"
-			(at 52.07 19.05 90)
-			(effects
-				(font
-					(size 1.27 1.27)
-				)
-			)
-		)
-		(property "Footprint" ""
-			(at 52.07 16.51 0)
+			(at 48.26 19.05 90)
+			(effects
+				(font
+					(size 1.27 1.27)
+				)
+			)
+		)
+		(property "Footprint" "TestPoint:TestPoint_Pad_D2.0mm"
+			(at 48.26 16.51 0)
 			(effects
 				(font
@@
 		)
 		(property "Datasheet" "~"
-			(at 52.07 16.51 0)
+			(at 48.26 16.51 0)
 			(effects
 				(font
@@
 		)
 		(property "Description" "test point"
-			(at 52.07 21.59 0)
+			(at 48.26 21.59 0)
 			(effects
 				(font
@@
 			(project ""
 				(path "/57b9e980-cd8f-44e4-af61-2cbd5bb30325/462ebe9c-fcaa-4c45-9d51-a2484be3186e"
-					(reference "TP3")
+					(reference "TP2")
 					(unit 1)
 				)
@@
 		(dnp no)
 		(fields_autoplaced yes)
-		(property "Reference" "U7"
+		(property "Reference" "U4"
 			(at 201.93 53.34 0)
 			(effects
@@
 			(project "ChipTester_354"
 				(path "/57b9e980-cd8f-44e4-af61-2cbd5bb30325/462ebe9c-fcaa-4c45-9d51-a2484be3186e"
-					(reference "U7")
+					(reference "U4")
 					(unit 1)
 				)
