File: KiCad/ChipTester_354.kicad_sch (KiCad schematic)
At the start: 9 parts

Commit message: Added milling machine files / updated schematic+pcb annotations /  updated footprints
Parts:
- renumbered D1 to D13, H3 to H1, H1 to H3, R1 to R11, S1 to S2
Changed lines of the file:
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@@
 		(dnp no)
 		(fields_autoplaced yes)
-		(property "Reference" "H1"
+		(property "Reference" "H3"
 			(at 34.29 115.5699 0)
 			(effects
@@
 			(project ""
 				(path "/57b9e980-cd8f-44e4-af61-2cbd5bb30325"
-					(reference "H1")
+					(reference "H3")
 					(unit 1)
 				)
@@
 		(dnp no)
 		(fields_autoplaced yes)
-		(property "Reference" "D1"
+		(property "Reference" "D13"
 			(at 115.57 63.8174 90)
 			(effects
@@
 			(project ""
 				(path "/57b9e980-cd8f-44e4-af61-2cbd5bb30325"
-					(reference "D1")
+					(reference "D13")
 					(unit 1)
 				)
@@
 		(dnp no)
 		(fields_autoplaced yes)
-		(property "Reference" "R1"
+		(property "Reference" "R11"
 			(at 114.3 55.8799 0)
 			(effects
@@
 			(project ""
 				(path "/57b9e980-cd8f-44e4-af61-2cbd5bb30325"
-					(reference "R1")
+					(reference "R11")
 					(unit 1)
 				)
@@
 		(dnp no)
 		(fields_autoplaced yes)
-		(property "Reference" "S1"
+		(property "Reference" "S2"
 			(at 96.52 48.26 0)
 			(effects
@@
 			(project ""
 				(path "/57b9e980-cd8f-44e4-af61-2cbd5bb30325"
-					(reference "S1")
+					(reference "S2")
 					(unit 1)
 				)
@@
 		(dnp no)
 		(fields_autoplaced yes)
-		(property "Reference" "H3"
+		(property "Reference" "H1"
 			(at 34.29 125.7299 0)
 			(effects
@@
 			(project "ChipTester_354"
 				(path "/57b9e980-cd8f-44e4-af61-2cbd5bb30325"
-					(reference "H3")
-					(unit 1)
-				)
+					(reference "H1")
+					(unit 1)
+				)
