File: KiCad_milling_machine/ChipTester_354.kicad_sch (KiCad schematic)
At the start: 9 parts

Commit message: Removed Switch
Other:
- sheet PWR Supply ports: added 4.5V, 4.5V VGND, 4.5V-; removed 4.5V/2.25V VGND, 4.5V/2.25V+, 4.5V/2.25V-
Changed lines of the file:
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@@
-			)
-		)
-		(pin "4.5V{slash}2.25V VGND" input
-			(at 144.78 40.64 180)
-			(effects
-				(font
-					(size 1.27 1.27)
-				)
-				(justify left)
 			)
 		)
@@
 			)
 		)
-		(pin "4.5V{slash}2.25V+" input
+		(pin "4.5V" input
 			(at 144.78 38.1 180)
 			(effects
@@
 			)
 		)
-		(pin "4.5V{slash}2.25V-" input
+		(pin "4.5V VGND" input
+			(at 144.78 40.64 180)
+			(effects
+				(font
+					(size 1.27 1.27)
+				)
+				(justify left)
+			)
+		)
+		(pin "4.5V-" input
 			(at 144.78 43.18 180)
 			(effects
