File: KiCad_milling_machine/pwrsup.kicad_sch (KiCad schematic)
At the start: 17 parts, among them U1 TLE2426xP, U2 L7805, U3 TLE2426xP, U4 TLE2426xP

Commit message: re-edited for 2nd milling, fixing clearances and problem areas
Parts:
- C2: value 0.33 µF -> 330 pF
- U2: footprint Package_TO_SOT_THT:TO-218-3_Horizontal_TabDown -> Package_TO_SOT_THT:TO-220-3_Horizontal_TabDown
Changed lines of the file:
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@@
 			)
 		)
-		(property "Footprint" "Package_TO_SOT_THT:TO-218-3_Horizontal_TabDown"
+		(property "Footprint" "Package_TO_SOT_THT:TO-220-3_Horizontal_TabDown"
 			(at 69.215 25.4 0)
 			(effects
@@
 			)
 		)
-		(property "Value" "0.33 µF"
+		(property "Value" "330 pF"
 			(at 58.42 31.7562 0)
 			(effects

Commit message: Removed Switch
Parts:
- removed C4: 1 µF, Capacitor_THT:CP_Radial_D5.0mm_P2.00mm, symbol Device:C_Small
- removed S2: 100SP3T2B4M6RE, 100SP3T2B4M6RE:100SP3T2B4M6RE, symbol 100SP3T2B4M6RE:100SP3T2B4M6RE
- removed TP6: 4.5/2.25V VGND, TestPoint:TestPoint_Pad_D2.0mm, symbol Connector:TestPoint_Small
- removed U3: TLE2426xP, Package_DIP:DIP-8_W7.62mm, symbol Reference_Voltage:TLE2426xP
Connections:
- net VBATT+ renamed 4.5V
- net VDIV renamed 4.5V VGND
Other:
- moved on the sheet: C5, TP7, U4
