File: KiCad_milling_machine/AD_INA.kicad_sch (KiCad schematic)
At the start: 8 parts

Commit message: Removed Switch
Connections:
- net REF: now also D3.2 (A), D5.2 (A); no longer D3.1 (K), D5.1 (K)
- net at D2.2 (A), R2.2: now also D3.1 (K); no longer D3.2 (A)
- net at D4.2 (A), R3.1: now also D5.1 (K); no longer D5.2 (A)
Other:
- moved on the sheet: D3, D5
Changed lines of the file:
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@@
 		(lib_id "Device:LED")
 		(at 68.58 88.9 90)
-		(unit 1)
-		(exclude_from_sim no)
-		(in_bom yes)
-		(on_board yes)
-		(dnp no)
-		(fields_autoplaced yes)
+		(mirror x)
+		(unit 1)
+		(exclude_from_sim no)
+		(in_bom yes)
+		(on_board yes)
+		(dnp no)
 		(property "Reference" "D5"
-			(at 72.39 89.2174 90)
+			(at 72.39 88.5826 90)
 			(effects
 				(font
@@
 		)
 		(property "Value" "WHT"
-			(at 72.39 91.7574 90)
+			(at 72.39 86.0426 90)
 			(effects
 				(font
@@
 		(lib_id "Device:LED")
 		(at 64.77 66.04 90)
-		(unit 1)
-		(exclude_from_sim no)
-		(in_bom yes)
-		(on_board yes)
-		(dnp no)
-		(fields_autoplaced yes)
+		(mirror x)
+		(unit 1)
+		(exclude_from_sim no)
+		(in_bom yes)
+		(on_board yes)
+		(dnp no)
 		(property "Reference" "D3"
-			(at 68.58 66.3574 90)
+			(at 68.58 65.7226 90)
 			(effects
 				(font
@@
 		)
 		(property "Value" "WHT"
-			(at 68.58 68.8974 90)
-			(effects
-				(font
+			(at 68.58 63.1826 90)
+			(effects
+				(font

Commit message: Ground inverting input of AD/INA circuit
Connections:
- net GND: now reaches U_T1.2 (-)
- no-connect marks 3 -> 2
Changed lines of the file:
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@@
-	)
-	(no_connect
-		(at 29.21 80.01)
 	)
 	(no_connect
@@
 	(wire
 		(pts
+			(xy 24.13 81.28) (xy 24.13 80.01)
+		)
+		(stroke
+			(width 0)
+			(type default)
+		)
+	)
+	(wire
+		(pts
 			(xy 76.2 53.34) (xy 76.2 71.12)
 		)
@@
 		(pts
 			(xy 36.83 104.14) (xy 36.83 92.71)
+		)
+		(stroke
+			(width 0)
+			(type default)
+		)
+	)
+	(wire
+		(pts
+			(xy 24.13 80.01) (xy 29.21 80.01)
 		)
 		(stroke
@@
 					(unit 1)
 				)
+			)
+		)
+	)
+	(symbol
+		(lib_id "power:GND")
+		(at 24.13 81.28 0)
+		(unit 1)
+		(exclude_from_sim no)
+		(in_bom yes)
+		(on_board yes)
+		(dnp no)
+		(fields_autoplaced yes)
+		(property "Reference" "#PWR09"
+			(at 24.13 87.63 0)
+			(effects
+				(font
+					(size 1.27 1.27)
+				)
+				(hide yes)
+			)
+		)
+		(property "Value" "GND"
+			(at 24.13 86.36 0)
+			(effects
+				(font
+					(size 1.27 1.27)
+				)
+			)
+		)
+		(property "Footprint" ""
+			(at 24.13 81.28 0)
+			(effects
+				(font
+					(size 1.27 1.27)
+				)
+				(hide yes)
+			)
+		)
+		(property "Datasheet" ""
+			(at 24.13 81.28 0)
+			(effects
+				(font
+					(size 1.27 1.27)
+				)
+				(hide yes)
+			)
+		)
+		(property "Description" "Power symbol creates a global label with name \"GND\" , ground"
+			(at 24.13 81.28 0)
+			(effects
+				(font
+					(size 1.27 1.27)
+				)
+				(hide yes)
+			)
+		)
+		(pin "1"
+		)
+		(instances
+			(project ""
+				(path "/57b9e980-cd8f-44e4-af61-2cbd5bb30325/2c721cfb-c552-4509-ae86-4c8bd0be2d45"
+					(reference "#PWR09")
+					(unit 1)
+				)

Commit message: grounded LEDs to allow for sufficient voltage blinking difference
Connections:
- net GND: now also D2.1 (K), D3.1 (K), D4.1 (K), D5.1 (K)
- net REF: no longer D2.1 (K), D3.2 (A), D4.1 (K), D5.2 (A)
- net at D2.2 (A), R2.2: now also D3.2 (A); no longer D3.1 (K)
- net at D4.2 (A), R3.1: now also D5.2 (A); no longer D5.1 (K)
Other:
- moved on the sheet: D3, D5
Changed lines of the file:
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@@
+	)
+	(junction
+		(at 76.2 71.12)
+		(diameter 0)
+		(color 0 0 0 0)
+	)
+	(junction
+		(at 80.01 93.98)
+		(diameter 0)
+		(color 0 0 0 0)
 	)
 	(junction
@@
 		)
 	)
-	(label "REFGND"
-		(at 76.2 71.12 90)
-		(effects
-			(font
-				(size 1.27 1.27)
-			)
-			(justify left bottom)
-		)
-	)
-	(label "REFGND"
-		(at 80.01 93.98 90)
-		(effects
-			(font
-				(size 1.27 1.27)
-			)
-			(justify left bottom)
-		)
-	)
 	(label "VS-"
 		(at 36.83 101.6 90)
@@
 			)
 			(justify right)
+		)
+	)
+	(symbol
+		(lib_id "power:GND")
+		(at 80.01 93.98 90)
+		(unit 1)
+		(exclude_from_sim no)
+		(in_bom yes)
+		(on_board yes)
+		(dnp no)
+		(fields_autoplaced yes)
+		(property "Reference" "#PWR010"
+			(at 86.36 93.98 0)
+			(effects
+				(font
+					(size 1.27 1.27)
+				)
+				(hide yes)
+			)
+		)
+		(property "Value" "GND"
+			(at 83.82 93.9799 90)
+			(effects
+				(font
+					(size 1.27 1.27)
+				)
+				(justify right)
+			)
+		)
+		(property "Footprint" ""
+			(at 80.01 93.98 0)
+			(effects
+				(font
+					(size 1.27 1.27)
+				)
+				(hide yes)
+			)
+		)
+		(property "Datasheet" ""
+			(at 80.01 93.98 0)
+			(effects
+				(font
+					(size 1.27 1.27)
+				)
+				(hide yes)
+			)
+		)
+		(property "Description" "Power symbol creates a global label with name \"GND\" , ground"
+			(at 80.01 93.98 0)
+			(effects
+				(font
+					(size 1.27 1.27)
+				)
+				(hide yes)
+			)
+		)
+		(pin "1"
+		)
+		(instances
+			(project "ChipTester_354"
+				(path "/57b9e980-cd8f-44e4-af61-2cbd5bb30325/2c721cfb-c552-4509-ae86-4c8bd0be2d45"
+					(reference "#PWR010")
+					(unit 1)
+				)
+			)
 		)
 	)
@@
 	(symbol
 		(lib_id "Device:LED")
-		(at 68.58 88.9 90)
+		(at 68.58 88.9 270)
 		(mirror x)
 		(unit 1)
@@
 		(dnp no)
 		(property "Reference" "D5"
-			(at 72.39 88.5826 90)
+			(at 64.77 89.2174 90)
 			(effects
 				(font
@@
 		)
 		(property "Value" "WHT"
-			(at 72.39 86.0426 90)
+			(at 64.77 91.7574 90)
 			(effects
 				(font
@@
 	(symbol
 		(lib_id "Device:LED")
-		(at 64.77 66.04 90)
+		(at 64.77 66.04 270)
 		(mirror x)
 		(unit 1)
@@
 		(dnp no)
 		(property "Reference" "D3"
-			(at 68.58 65.7226 90)
+			(at 60.96 66.3574 90)
 			(effects
 				(font
@@
 		)
 		(property "Value" "WHT"
-			(at 68.58 63.1826 90)
+			(at 60.96 68.8974 90)
 			(effects
 				(font
@@
 					(unit 1)
 				)
+			)
+		)
+	)
+	(symbol
+		(lib_id "power:GND")
+		(at 76.2 71.12 90)
+		(unit 1)
+		(exclude_from_sim no)
+		(in_bom yes)
+		(on_board yes)
+		(dnp no)
+		(fields_autoplaced yes)
+		(property "Reference" "#PWR011"
+			(at 82.55 71.12 0)
+			(effects
+				(font
+					(size 1.27 1.27)
+				)
+				(hide yes)
+			)
+		)
+		(property "Value" "GND"
+			(at 80.01 71.1199 90)
+			(effects
+				(font
+					(size 1.27 1.27)
+				)
+				(justify right)
+			)
+		)
+		(property "Footprint" ""
+			(at 76.2 71.12 0)
+			(effects
+				(font
+					(size 1.27 1.27)
+				)
+				(hide yes)
+			)
+		)
+		(property "Datasheet" ""
+			(at 76.2 71.12 0)
+			(effects
+				(font
+					(size 1.27 1.27)
+				)
+				(hide yes)
+			)
+		)
+		(property "Description" "Power symbol creates a global label with name \"GND\" , ground"
+			(at 76.2 71.12 0)
+			(effects
+				(font
+					(size 1.27 1.27)
+				)
+				(hide yes)
+			)
+		)
+		(pin "1"
+		)
+		(instances
+			(project "ChipTester_354"
+				(path "/57b9e980-cd8f-44e4-af61-2cbd5bb30325/2c721cfb-c552-4509-ae86-4c8bd0be2d45"
+					(reference "#PWR011")
+					(unit 1)
+				)
